Commit message: Implement comprehensive thumb pinching fix for DexPilot system
- Added final validation test script (final_validation_test.py) to validate the complete thumb pinching fix system, including component initialization, validation scenarios, and hardware integration tests.
- Developed targeted thumb pinching fix module (fix_thumb_pinching.py) to analyze thumb motion issues and implement corrective strategies.
- Created integrated testing script (test_integrated_thumb_correction.py) to simulate and validate the thumb pinch correction within the DexPilot processing pipeline.
- Introduced thumb pinch corrector class (thumb_pinch_corrector.py) to provide real-time corrections during pinching gestures, addressing the identified thumb drop issue.
- Enhanced hardware mapping tests to ensure accurate translation of URDF joint angles to hardware commands.

File: assets/unitree_hand/unitree_dex3_left.urdf (robot description, URDF)
Before this commit: robot dex3_left, 15 links, 14 joints
Joints:
- joint left_hand_thumb_1_joint: limit lower=-0.72431163 upper=0.920 effort=1.4 velocity=12 -> lower=-0.72431163 upper=1.22 effort=1.4 velocity=12

File: assets/unitree_hand/unitree_dex3_right.urdf (robot description, URDF)
Before this commit: robot dex3_right, 15 links, 14 joints
Joints:
- joint right_hand_thumb_1_joint: limit lower=-0.920 upper=0.72431163 effort=1.4 velocity=12 -> lower=-0.72431163 upper=1.22 effort=1.4 velocity=12

Commit message: refactor: change hand urdf files back to original

File: assets/unitree_hand/unitree_dex3_left.urdf (robot description, URDF)
Before this commit: robot dex3_left, 15 links, 14 joints
Joints:
- joint left_hand_thumb_1_joint: limit lower=-0.72431163 upper=1.22 effort=1.4 velocity=12 -> lower=-0.72431163 upper=0.920 effort=1.4 velocity=12

File: assets/unitree_hand/unitree_dex3_right.urdf (robot description, URDF)
Before this commit: robot dex3_right, 15 links, 14 joints
Joints:
- joint right_hand_thumb_1_joint: limit lower=-0.72431163 upper=1.22 effort=1.4 velocity=12 -> lower=-0.920 upper=0.72431163 effort=1.4 velocity=12

Commit message: theory: Problem was caused by mismatch between thumb_0 angles in urdf and new hand after update

File: assets/unitree_hand/unitree_dex3_left.urdf (robot description, URDF)
Before this commit: robot dex3_left, 15 links, 14 joints
Joints:
- joint left_hand_thumb_0_joint: limit lower=-1.04719755 upper=1.04719755 effort=2.45 velocity=6.857 -> lower=-2.094395 upper=0 effort=2.45 velocity=6.857

Commit message: feat: adjust joint limits and refine target angles for thumb pinching dynamics

File: assets/unitree_hand/unitree_dex3_left.urdf (robot description, URDF)
Before this commit: robot dex3_left, 15 links, 14 joints
Joints:
- joint left_hand_thumb_0_joint: limit lower=-2.094395 upper=0 effort=2.45 velocity=6.857 -> lower=-2.443461 upper=0.174533 effort=2.45 velocity=6.857
